File: Electronic Design/SAO Voja4 Adapter V1.0/SAO Voja4 Adapter.kicad_pcb (KiCad board)
At the start: 2 copper layers, 38.1 x 50.8 mm, 39 parts, among them J1 Conn_01x12_Socket, J2 BATTERY, Q1 MMBT4401LT1G, Q2 MMBT4401LT1G, Q3 MMBT4401LT1G, Q4 MMBT4401LT1G, U1 SSP9193-33M5R, X1 SAO_conn, X2 Header_11-PIN_0.1, X3 HEADER_11-PIN_0.1, X4 QWIIC

Commit message: Released V1 boards
Parts:
- removed kibuzzard-66D35F07: G***, kibuzzard-66D35F07
- removed kibuzzard-67170228: G***, kibuzzard-67170228
- added kibuzzard-671724A5: G***, kibuzzard-671724A5, F.Cu at (107.5, 151.0)
- J1: footprint Connector_PinSocket_2.54mm:PinSocket_1x12_P2.54mm_Horizontal -> Andy_Footprint_Library:PinSocket_1x12_P2.54mm_Horizontal_Overhang
- L1: moved to B.Cu
- X2: value Header_11-PIN_0.1 -> Header_9-PIN_0.1; footprint Connector_PinSocket_2.54mm:PinSocket_1x11_P2.54mm_Vertical -> Connector_PinSocket_2.54mm:PinSocket_1x09_P2.54mm_Vertical
- moved L1 39.8 mm to (120.5, 130.5), turned to 180 degrees
- moved JP10 27.4 mm to (118.9, 146.6)
- moved JP23 25.6 mm to (92.3, 146.7)
- moved JP2 23.2 mm to (118.9, 141.3)
- moved JP4 20.6 mm to (112.7, 141.3)
- moved JP11 20.3 mm to (115.1, 146.6)
- moved R2 20.1 mm to (118.9, 128.8), turned to -90 degrees
- moved Q1 18.7 mm to (118.9, 132.7), turned to 90 degrees
- moved JP22 18.6 mm to (96.1, 146.7)
- moved C3 18.2 mm to (124.5, 117.5), turned to 180 degrees
- moved Q4 14.9 mm to (99.9, 132.7), turned to 90 degrees
- moved U1 14.0 mm to (124.5, 125.8), turned to 90 degrees
- moved JP12 13.5 mm to (111.3, 146.6)
- moved R6 12.7 mm to (99.9, 128.8), turned to -90 degrees
- moved JP21 11.9 mm to (99.9, 146.7)
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- renumbered JP3 to JP2, JP4 to JP3, JP2 to JP4, R5 to R1, R1 to R2, R2 to R3, R6 to R5, R7 to R6
Connections:
- JP11 pad 2: /SPI_CS1 -> /SPI_CS
- JP2 pad 2: /OUT0 -> /jOUT0
- JP30 pad 2: /SPI_CS1 -> /SPI_CS
- JP4 pad 2: /OUT1 -> /jOUT1
- R1 pad 2: /OUT0 -> /jOUT0
- R4 pad 2: /OUT1 -> /jOUT1
- X2 pad 1: /SPI_CS2 -> /SPI_CD
- X2 pad 2: /SPI_RST -> unconnected-(X2-Pin_2-Pad2)
- X2 pad 3: /SPI_CD -> unconnected-(X2-Pin_3-Pad3)
- X2 pad 4: /QSPI_D2 -> /SPI_CS1
- X2 pad 5: /QSPI_D1 -> /SPI_SDO
- X2 pad 6: /SPI_CS1 -> /SPI_SDI
- X2 pad 7: /SPI_SDO -> /SPI_CLK
- X2 pad 8: /SPI_SDI -> GND
- X2 pad 9: /SPI_CLK -> VIN
Routing:
- net GND: track 0.00 -> 142.0 mm, vias 0 -> 11
- net VIN: track 0.00 -> 115.2 mm, vias 0 -> 8
- net /OUT2: track 0.00 -> 74.3 mm, vias 0 -> 1
- net /IN2: track 0.00 -> 67.8 mm, vias 0 -> 1
- net /OUT3: track 0.00 -> 64.0 mm, vias 0 -> 3
- net /IN3: track 0.00 -> 52.6 mm, vias 0 -> 4
- net /SAO_SDA: track 0.00 -> 51.5 mm, vias 0 -> 3
- net /SPI_DC: track 0.00 -> 50.9 mm, vias 0 -> 2
- net /SPI_SDI: track 0.00 -> 47.5 mm, vias 0 -> 2
- net /SPI_CLK: track 0.00 -> 45.9 mm, vias 0 -> 2
- net /SPI_SDO: track 0.00 -> 44.8 mm, vias 0 -> 2
- net /SPI_CD: track 0.00 -> 43.6 mm, vias 0 -> 2
- net /SAO_SCL: track 0.00 -> 42.1 mm
- net /SPI_CS: track 0.00 -> 37.1 mm, vias 0 -> 2
- net /SPI_CS1: track 0.00 -> 31.3 mm, vias 0 -> 3
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Other:
- board text added: "0"
- board text added: "1"
- board text added: "3V3"
- board text added: "Alt. Bat."
- board text added: "CD"
- board text added: "CLK"
- board text added: "CS"
- board text added: "CS1"
- board text added: "CS2"
- board text added: "DC"
- board text added: "Exclusively for the VOJA4 BADGE from Supercon.6 (2022)"
- board text added: "GND"
- board text added: "GPIO1"
- board text added: "GPIO2"
- board text added: "I2C ZONE"
- board text added: "IN"
- board text added: "IN2"
- board text added: "IN3"
- board text added: "OLED"
- board text added: "OUT"
- board text added: "OUT2"
- board text added: "OUT3"
- board text added: "QWIIC"
- board text added: "RST"
- board text added: "SAO"
- board text added: "SD"
- board text added: "SDI"
- board text added: "SDO"
- board text added: "SPI ZONE"
- board text added: "VIN"
- board text added: "X"
- board text added: "www.MachineIdeas.com Designed by Andy Geppert In collaboration with Koppany Horvath"
- board text added: "www.adafruit.com/product/1431"
- board text added: "www.adafruit.com/product/4682"
- board text added: "www.hackaday.io/project/188025"
- board text added: "www.hackaday.io/project/198394"
- board text removed: "www.Core64.io Andy Geppert"
